Commit message: Able to display and see the turtle bot now

File: nuturtle_description/urdf/turtlebot3_burger.urdf.xacro (robot description, xacro)
@@ -13,5 +13,5 @@
       <origin xyz="-0.032 0 0.0" rpy="0 0 0"/>
       <geometry>
-        <mesh filename="${find nuturtle_description)/mesh/burger_base.stl" scale="0.001 0.001 0.001"/>
+        <mesh filename="file://$(find nuturtle_description)/mesh/burger_base.stl" scale="0.001 0.001 0.001"/>
       </geometry>
       <material name="light_black"/>
@@ -39,5 +39,5 @@
       <origin xyz="0 0 0" rpy="1.57 0 0"/>
       <geometry>
-        <mesh filename="${find nuturtle_description)/mesh/left_tire.stl" scale="0.001 0.001 0.001"/>
+        <mesh filename="file://$(find nuturtle_description)/mesh/left_tire.stl" scale="0.001 0.001 0.001"/>
       </geometry>
       <material name="dark"/>
@@ -65,5 +65,5 @@
       <origin xyz="0 0 0" rpy="1.57 0 0"/>
       <geometry>
-        <mesh filename="${find nuturtle_description)/mesh/right_tire.stl" scale="0.001 0.001 0.001"/>
+        <mesh filename="file://$(find nuturtle_description)/mesh/right_tire.stl" scale="0.001 0.001 0.001"/>
       </geometry>
       <material name="dark"/>
@@ -114,5 +114,5 @@
       <origin xyz="0 0 0.0" rpy="0 0 0"/>
       <geometry>
-        <mesh filename="${find nuturtle_description)/mesh/lds.stl" scale="0.001 0.001 0.001"/>
+        <mesh filename="file://$(find nuturtle_description)/mesh/lds.stl" scale="0.001 0.001 0.001"/>
       </geometry>
       <material name="dark"/>

Commit message: Task A.3 working

File: nuturtle_description/urdf/turtlebot3_burger.urdf.xacro (robot description, xacro)
@@ -3,4 +3,9 @@
   xmlns:xacro="http://ros.org/wiki/xacro">
   <xacro:include filename="$(find nuturtle_description)/urdf/common_properties.urdf"/>
+  <xacro:property name="yaml_file" value="$(find nuturtle_description)/config/diff_params.yaml" />
+  <xacro:property name="ddrive_prop" value="${xacro.load_yaml(yaml_file)['/**']['ros__parameters']}" />
+  <xacro:property name="wheel_radius" value="${ddrive_prop['wheel_radius']}" />
+  <xacro:property name="track_width" value="${ddrive_prop['track_width']}" />
+  <xacro:property name="collision_radius" value="${ddrive_prop['collision_radius']}" />
   <link name="base_footprint"/>
   <joint name="base_joint" type="fixed">
@@ -20,5 +25,10 @@
       <origin xyz="-0.032 0 0.070" rpy="0 0 0"/>
       <geometry>
-        <box size="0.140 0.140 0.143"/>
+        <xacro:if value = "${collision_radius &gt; 0}">
+          <cylinder radius="${collision_radius}" length = "0.143" />
+        </xacro:if>
+        <xacro:if value = "${not collision_radius &gt; 0}">
+          <box size="0.140 0.140 0.143"/>
+        </xacro:if>
       </geometry>
     </collision>
@@ -32,5 +42,5 @@
     <parent link="base_link"/>
     <child link="wheel_left_link"/>
-    <origin xyz="0.0 0.08 0.023" rpy="-1.57 0 0"/>
+    <origin xyz="0.0 ${track_width/2} 0.023" rpy="-1.57 0 0"/>
     <axis xyz="0 0 1"/>
   </joint>
@@ -46,5 +56,5 @@
       <origin xyz="0 0 0" rpy="0 0 0"/>
       <geometry>
-        <cylinder length="0.018" radius="0.033"/>
+        <cylinder length="0.018" radius="${wheel_radius}"/>
       </geometry>
     </collision>
@@ -58,5 +68,5 @@
     <parent link="base_link"/>
     <child link="wheel_right_link"/>
-    <origin xyz="0.0 -0.080 0.023" rpy="-1.57 0 0"/>
+    <origin xyz="0.0 -${track_width/2} 0.023" rpy="-1.57 0 0"/>
     <axis xyz="0 0 1"/>
   </joint>
@@ -72,5 +82,5 @@
       <origin xyz="0 0 0" rpy="0 0 0"/>
       <geometry>
-        <cylinder length="0.018" radius="0.033"/>
+        <cylinder length="0.018" radius="${wheel_radius}"/>
       </geometry>
     </collision>

Commit message: Task A4 able to do purple but missing fixed-frame setting and other colors

File: nuturtle_description/urdf/turtlebot3_burger.urdf.xacro (robot description, xacro)
@@ -8,4 +8,7 @@
   <xacro:property name="track_width" value="${ddrive_prop['track_width']}" />
   <xacro:property name="collision_radius" value="${ddrive_prop['collision_radius']}" />
+  <!-- Possible value red green blue purple -->
+  <xacro:property name="color" value="$(arg color)" />
+  <!-- <xacro:property name="color" value="red" /> -->
   <link name="base_footprint"/>
   <joint name="base_joint" type="fixed">
@@ -20,5 +23,5 @@
         <mesh filename="file://$(find nuturtle_description)/mesh/burger_base.stl" scale="0.001 0.001 0.001"/>
       </geometry>
-      <material name="light_black"/>
+      <material name="${color}"/>
     </visual>
     <collision>

Commit message: Have a very basic version of launch file written

File: nuturtle_description/urdf/turtlebot3_burger.urdf.xacro (robot description, xacro)
@@ -15,4 +15,6 @@
   <xacro:property name="track_width" value="${ddrive_prop['track_width']}" />
   <xacro:property name="collision_radius" value="${ddrive_prop['collision_radius']}" />
+  <xacro:property name="wheel_left_name" value="${ddrive_prop['wheel_left']}" />
+  <xacro:property name="wheel_right_name" value="${ddrive_prop['wheel_right']}" />
   <!-- Possible value red green blue purple -->
   <xacro:property name="color" value="$(arg color)" />
@@ -49,5 +51,5 @@
     </inertial>
   </link>
-  <joint name="wheel_left_joint" type="continuous">
+  <joint name="${wheel_left_name}" type="continuous">
     <parent link="base_link"/>
     <child link="wheel_left_link"/>
@@ -75,5 +77,5 @@
     </inertial>
   </link>
-  <joint name="wheel_right_joint" type="continuous">
+  <joint name="${wheel_right_name}" type="continuous">
     <parent link="base_link"/>
     <child link="wheel_right_link"/>
